Commit message: Prefer no space before closing xml />

File: uwreact_description/urdf/common/simple_shapes.xacro (robot description, xacro)
@@ -9,10 +9,10 @@
       <inertia ixx="${mass * (ly*ly + lz*lz) / 12}"  ixy="0"  ixz="0"
                 iyy="${mass * (lx*lx + lz*lz) / 12}" iyz="0"
-                izz="${mass * (lx*lx + ly*ly) / 12}" />
+                izz="${mass * (lx*lx + ly*ly) / 12}"/>
     </inertial>
       <visual>
       <origin xyz="${xyz}" rpy="${rpy}"/>
       <geometry>
-        <box size="${lx} ${ly} ${lz}" />
+        <box size="${lx} ${ly} ${lz}"/>
       </geometry>
       <material name="${color}"/>
@@ -21,5 +21,5 @@
       <origin xyz="${xyz}" rpy="${rpy}"/>
       <geometry>
-        <box size="${lx} ${ly} ${lz}" />
+        <box size="${lx} ${ly} ${lz}"/>
       </geometry>
     </collision>
@@ -37,10 +37,10 @@
       <inertia ixx="${mass * (3*rad*rad + len*len) / 12}"  ixy="0"  ixz="0"
                 iyy="${mass * (3*rad*rad + len*len) / 12}" iyz="0"
-                izz="${mass * rad*rad / 2}" />
+                izz="${mass * rad*rad / 2}"/>
     </inertial>
       <visual>
         <origin xyz="${xyz}" rpy="${rpy}"/>
         <geometry>
-          <cylinder length="${len}" radius="${rad}" />
+          <cylinder length="${len}" radius="${rad}"/>
         </geometry>
       <material name="${color}"/>
@@ -49,5 +49,5 @@
         <origin xyz="${xyz}" rpy="${rpy}"/>
         <geometry>
-          <cylinder length="${len}" radius="${rad}" />
+          <cylinder length="${len}" radius="${rad}"/>
         </geometry>
     </collision>
